File: hw/R2P_GW_module.sch (EAGLE design)
At the start: 32 parts, among them U1 STM32F103CX, U5 LD3985XX, X1 MICROMATCH-4

Commit message: First PCB version almost finished
Andrea Zoppi
Parts:
- removed SOT1: MAX3051, maxim:MAX3051
- removed U$1: ASE, crystal:ASE
- removed U5: LD3985XX, st:LD3985XX
- added C10, C13, C14, C15, C16, C17, C22, C23, C25, C26, C27, C8: 100n, rcl:C-EUC0603
- added C12: 4u7, rcl:C-EUC0805
- added C2, C3: 2u2, rcl:C-EUC0805
- added C24: 10u, rcl:C-EUC0805
- added C28: 15p, rcl:C-EUC0603
- added C4: 1u, rcl:C-EUC0805
- added OSC1: ASE 8MHz, crystal:ASE
- added OSC2: ASE 50MHz, crystal:ASE
- added R10, R15, R7: 2k2, rcl:R-EU_R0603
- added R11, R14: 22, rcl:R-EU_R0603
- added R12: 100k, rcl:R-EU_R0603
- added R13: 1k5, rcl:R-EU_R0603
- added R5: 47, rcl:R-EU_R0603
- added R6: 4k87, rcl:R-EU_R0603
- added R8, R9: 220, rcl:R-EU_R0603
- added RN1, RN3, RN5: 51, resistor-dil:4R-NCAT16
- added RN2, RN4: 2k2, resistor-dil:4R-NCAT16
- added U2: DP83848C, texas-instruments:DP83848C
- added U3: LD3985XX, st:LD3985XX
- added U4: MAX3051, maxim:MAX3051
- added X2: 47589-0001, molex:47589-0001
- added X3: (no value), bel:SI-60062-F
- C11: value 15pF -> 15p
- C21: value 4.7u -> 4u7
- R2: value 10k -> 100k
- U1: value STM32F103CX -> STM32F407VG; device st:STM32F103CX -> st:STM32F407VG
Connections:
- removed net AM_DRDY: U1.PB5
- removed net AM_INT1: U1.PB6
- removed net AM_INT2: U1.PB7
- removed net BOOT0: R2.2, U1.BOOT0
- removed net GPS_RESET: U1.PA4
- removed net GPS_RX: U1.PA3
- removed net GPS_STATUS: U1.PA1
- removed net GPS_TX: U1.PA2
- removed net GYRO_CS: U1.PB0
- removed net GYRO_INT1: U1.PB10
- removed net GYRO_INT2: U1.PB1
- removed net MISO: U1.PA6
- removed net MOSI: U1.PA7
- removed net NRST: U$4.P$10, U1.NRST
- removed net OSC_IN: U$1.OUT, U1.PD0/OSC_IN
- removed net OSC_OUT: U1.PD1/OSC_OUT
- removed net SCK: U1.PA5
- removed net SCL: U1.PB8
- removed net SDA: U1.PB9
- new net !ETH_PWRDN: OSC2.TRI, RN4C.2, U2.!PWRDOWN!/INT
- new net !RESET: R15.1, RN2A.1, U$4.10, U1IO.NRST, U2.!RESET
- new net ETH_RMII_CRS_DV: RN5B.1, U1IO.PA7
- new net ETH_RMII_MDC: U1IO.PC1, U2.MDC
- new net ETH_RMII_MDIO: R13.1, U1IO.PA2, U2.MDIO
- new net ETH_RMII_REF_CLK: OSC2.OUT, U1IO.PA1, U2.X1
- new net ETH_RMII_RXD0: RN5C.1, U1IO.PC4
- new net ETH_RMII_RXD1: RN5D.1, U1IO.PC5
- new net ETH_RMII_TXD0: RN3C.1, U1IO.PB12
- new net ETH_RMII_TXD1: RN3D.1, U1IO.PB13
- new net ETH_RMII_TXEN: RN3B.1, U1IO.PB11
- new net MCU_CLK: OSC1.OUT, U1IO.PH0
- new net N$10: RN1C.1, U2.RX+, X3.RD+
- new net N$11: RN1D.1, U2.RX-, X3.RD-
- new net N$12: R9.2, X3.YA
- new net N$13: C14.2, X3.CT
- new net N$14: C17.1, C22.1, C23.1, C24.1, U2.PFBIN1, U2.PFBIN2, U2.PFBOUT
- new net N$16: C16.2, X3.CR
- new net N$17: R8.2, X3.GA
- new net N$19: RN2C.1, U2.LED_SPEED/AN1
- new net N$21: RN3B.2, U2.TX_EN
- new net N$23: RN2B.1, U2.LED_LINK/AN0, X3.YK
- new net N$24: RN2D.1, U2.LED_ACT/COL/LAN_EN, X3.GK
- new net N$25: RN3C.2, U2.TX_D0
- new net N$26: R2.1, U1IO.BOOT0
- new net N$27: R7.1, U2.RESERVED_PU1
- new net N$28: R10.1, U2.RESERVED_PU2
- new net N$29: RN3D.2, U2.TX_D1
- new net N$30: RN4A.2, U2.TX_D2
- new net N$31: RN4B.2, U2.TX_D3/SNI_MODE
- new net N$32: R14.2, X2.3
- new net N$34: RN5C.2, U2.RX_D0/PHYAD1
- new net N$38: R12.1, U2.RX_DV/MII_MODE
- new net N$40: RN5D.2, U2.RX_D1/PHYAD2
- new net N$41: RN5B.2, U2.CRS/CRS_DV/LED_CFG
- new net N$6: R6.1, U2.RBIAS
- new net N$7: R11.2, X2.2
- new net N$8: RN1A.1, U2.TX+, X3.TD+
- new net N$9: RN1B.1, U2.TX-, X3.TD-
- new net USB_DM: R11.1, U1IO.PA11
- new net USB_DP: R14.1, U1IO.PA12
- new net USB_ID: U1IO.PA10, X2.4
- new net USB_VBUS: U1IO.PA9, X2.1
- new net VCAP_1: C3.1, U1PWR.VCAP_1
- new net VCAP_2: C2.1, U1PWR.VCAP_2
- net +3V3: now also C10.1, C12.1, C13.1, C15.1, C25.1, C26.1, C27.1, C28.1, OSC1.VDD, OSC2.VDD, R10.2, R12.2, R13.2, R15.2, R5.2, R7.2, R8.1, R9.1, RN1A.2, RN1B.2, RN1C.2, RN1D.2, RN2A.2, RN2B.2, RN2C.2, RN2D.2, RN4C.1, U$4.1, U1PWR.VBAT, U1PWR.VDD, U1PWR.VDDA, U1PWR.VDD_1, U1PWR.VDD_12, U1PWR.VDD_2, U1PWR.VDD_4, U1PWR.VDD_5, U2.AVDD33, U2.IOVDD33-1, U2.IOVDD33-2, U3.VOUT, U4.VCC; no longer SOT1.VCC, U$1.VDD, U$4.P$1, U1.VBAT, U1.VDD_1, U1.VDD_2, U1.VDD_3, U1.VDD_A, U5.VOUT
- net CANH: now also U4.CANH; no longer SOT1.CANH
- net CANL: now also U4.CANL; no longer SOT1.CANL
- net CAN_RX: now also U1IO.PD0, U4.RXD; no longer SOT1.RXD, U1.PA11
- net CAN_TX: now also U1IO.PD1, U4.TXD; no longer SOT1.TXD, U1.PA12
- net GND: now also C10.2, C12.2, C13.2, C14.1, C15.2, C16.1, C17.2, C2.2, C22.2, C23.2, C24.2, C25.2, C26.2, C27.2, C28.2, C3.2, C4.2, C8.2, OSC1.GND, OSC2.GND, R2.2, R6.2, RN3A.1, RN3A.2, RN4A.1, RN4B.1, RN4D.1, RN4D.2, RN5A.1, RN5A.2, U$4.3, U$4.5, U$4.9, U1PWR.VSS, U1PWR.VSSA, U1PWR.VSS_2, U1PWR.VSS_4, U1PWR.VSS_5, U2.AGND1, U2.AGND2, U2.DGND, U2.IOGND1, U2.IOGND2, U3.GND, U4.GND, X2.5, X2.SHLD1, X2.SHLD2, X2.SHLD3, X2.SHLD4, X3.8, X3.SHLD1, X3.SHLD2; no longer R2.1, SOT1.GND, U$1.GND, U$4.P$3, U$4.P$9, U1.VSS_1, U1.VSS_2, U1.VSS_3, U1.VSS_A, U5.GND
- net JTCK: now also U$4.4, U1IO.PA14; no longer U$4.P$4, U1.PA14
- net JTDI: now also U$4.8, U1IO.PA15; no longer U$4.P$8, U1.PA15
- net JTDO: now also U$4.6, U1IO.PB3; no longer U$4.P$6, U1.PB3
- net JTMS: now also U$4.2, U1IO.PA13; no longer U$4.P$2, U1.PA13
- net LED1: no longer U1.PB12
- net LED2: no longer U1.PB13
- net LED3: no longer U1.PB14
- net LED4: no longer U1.PB15
- net N$1: now also C4.1, C8.1, R5.1, U1PWR.VREF+; no longer U$4.P$5
- net N$2: now also U4.RS; no longer SOT1.RS
- net N$3: now also OSC1.TRI; no longer U$1.TRI
- net N$4: now also U3.BYPASS; no longer U5.BYPASS
- net N$5: now also U3.INHIBIT, U3.VIN; no longer U5.INHIBIT, U5.VIN
- net UART_RX: now also U1IO.PB7; no longer U1.PA10
- net UART_TX: now also U1IO.PB6; no longer U1.PA9
Other:
- note added: "CAN BUS DRIVER"
- note added: "CAN BUS INTERFACE"
- note added: "ETHERNET TRANSCEIVER AND INTERFACE"
- note added: "MCU"
- note added: "MCU CLOCK"
- note added: "MCU POWER"
- note added: "POWER SUPPLY"
- note added: "UART INTERFACE"
- note added: "USB INTERFACE"
- note removed: "BUS CONNECTORS"
- note removed: "POWER SUPPLY AND CAN BUS DRIVER"
- note removed: "STM32"
- moved on the sheet: C1, C11, C18, C19, C20, C21, C5, C6, C7, C9, JP1, JP2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

Commit message: All the PCB elements routed
The board has yet to be finally checked.

Andrea Zoppi
Connections:
- net !ETH_PWRDN: now also U1IO.PC3
- net LED1: now also U1IO.PC10
- net LED2: now also U1IO.PC11
- net LED3: now also U1IO.PB8
- net LED4: now also U1IO.PB9
Changed lines of the file:
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@@
 <wire x1="152.4" y1="71.12" x2="154.94" y2="71.12" width="0.1524" layer="91"/>
+</segment>
+<segment>
+<pinref part="U1" gate="IO" pin="PC10"/>
+<wire x1="60.96" y1="137.16" x2="63.5" y2="137.16" width="0.1524" layer="91"/>
+<label x="60.96" y="137.16" size="1.778" layer="95" rot="MR0"/>
 </segment>
 </net>
@@
 <pinref part="R22" gate="G$1" pin="1"/>
 </segment>
+<segment>
+<pinref part="U1" gate="IO" pin="PB8"/>
+<wire x1="60.96" y1="185.42" x2="63.5" y2="185.42" width="0.1524" layer="91"/>
+<label x="60.96" y="185.42" size="1.778" layer="95" rot="MR0"/>
+</segment>
 </net>
 <net name="LED2" class="0">
@@
 <pinref part="R19" gate="G$1" pin="1"/>
 </segment>
+<segment>
+<pinref part="U1" gate="IO" pin="PC11"/>
+<wire x1="60.96" y1="134.62" x2="63.5" y2="134.62" width="0.1524" layer="91"/>
+<label x="60.96" y="134.62" size="1.778" layer="95" rot="MR0"/>
+</segment>
 </net>
 <net name="LED4" class="0">
@@
 <label x="154.94" y="63.5" size="1.778" layer="95"/>
 <pinref part="R18" gate="G$1" pin="1"/>
+</segment>
+<segment>
+<pinref part="U1" gate="IO" pin="PB9"/>
+<wire x1="60.96" y1="182.88" x2="63.5" y2="182.88" width="0.1524" layer="91"/>
+<label x="60.96" y="182.88" size="1.778" layer="95" rot="MR0"/>
 </segment>
 </net>
@@
 <junction x="193.04" y="226.06"/>
 </segment>
-</net>
+<segment>
+<pinref part="U1" gate="IO" pin="PC3"/>
+<wire x1="60.96" y1="154.94" x2="63.5" y2="154.94" width="0.1524" layer="91"/>
+<label x="60.96" y="154.94" size="1.778" layer="95" rot="MR0"/>
+</segment>
+</net>

Commit message: Minor refinements
Andrea Zoppi
Parts:
- C4: device rcl:C-EUC0805 -> rcl:C-EUC0603
Other:
- moved on the sheet: X1-2
Changed lines of the file:
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@@
 <part name="GND3" library="supply1" deviceset="GND" device=""/>
 <part name="GND10" library="supply1" deviceset="GND" device=""/>
-<part name="C4" library="rcl" deviceset="C-EU" device="C0805" value="1u"/>
 <part name="C8" library="rcl" deviceset="C-EU" device="C0603" value="100n"/>
 <part name="GND13" library="supply1" deviceset="GND" device=""/>
@@
 <part name="+3V12" library="supply1" deviceset="+3V3" device=""/>
 <part name="C18" library="rcl" deviceset="C-EU" device="C0603" value="100n"/>
+<part name="C4" library="rcl" deviceset="C-EU" device="C0603" value="1u"/>
 </parts>
 <sheets>
@@
 <instance part="R3" gate="G$1" x="223.52" y="76.2" rot="R180"/>
 <instance part="R4" gate="G$1" x="185.42" y="35.56" rot="R90"/>
-<instance part="GND8" gate="1" x="264.16" y="20.32"/>
+<instance part="GND8" gate="1" x="264.16" y="15.24"/>
 <instance part="P+1" gate="1" x="88.9" y="43.18"/>
 <instance part="P+2" gate="1" x="129.54" y="43.18"/>
@@
 <instance part="X1" gate="-1" x="256.54" y="33.02" smashed="yes">
 <attribute name="NAME" x="256.032" y="33.782" size="1.524" layer="95" rot="R180"/>
-<attribute name="VALUE" x="256.54" y="13.589" size="1.778" layer="96"/>
+<attribute name="VALUE" x="250.571" y="15.24" size="1.778" layer="96" rot="R90"/>
 </instance>
-<instance part="X1" gate="-2" x="256.54" y="30.48"/>
+<instance part="X1" gate="-2" x="256.54" y="20.32"/>
 <instance part="X1" gate="-3" x="256.54" y="27.94"/>
 <instance part="X1" gate="-4" x="256.54" y="25.4"/>
@@
 <instance part="GND3" gate="1" x="312.42" y="50.8"/>
 <instance part="GND10" gate="1" x="320.04" y="50.8"/>
-<instance part="C4" gate="G$1" x="365.76" y="78.74"/>
 <instance part="C8" gate="G$1" x="373.38" y="78.74"/>
 <instance part="GND13" gate="1" x="365.76" y="71.12"/>
@@
 <instance part="GND39" gate="1" x="106.68" y="137.16"/>
 <instance part="X2" gate="X" x="99.06" y="81.28"/>
-<instance part="P+3" gate="1" x="264.16" y="40.64"/>
+<instance part="P+3" gate="1" x="264.16" y="43.18"/>
 <instance part="P+4" gate="1" x="185.42" y="45.72"/>
 <instance part="OSC1" gate="G$1" x="203.2" y="81.28"/>
@@
 <instance part="+3V12" gate="G$1" x="101.6" y="172.72"/>
 <instance part="C18" gate="G$1" x="269.24" y="83.82"/>
+<instance part="C4" gate="G$1" x="365.76" y="78.74"/>
 </instances>
 <busses>
@@
 </segment>
 <segment>
-<wire x1="261.62" y1="30.48" x2="264.16" y2="30.48" width="0.1524" layer="91"/>
-<wire x1="264.16" y1="30.48" x2="264.16" y2="22.86" width="0.1524" layer="91"/>
+<wire x1="261.62" y1="20.32" x2="264.16" y2="20.32" width="0.1524" layer="91"/>
+<wire x1="264.16" y1="20.32" x2="264.16" y2="17.78" width="0.1524" layer="91"/>
 <pinref part="GND8" gate="1" pin="GND"/>
 <pinref part="X1" gate="-2" pin="S"/>
@@
 </segment>
 <segment>
-<pinref part="C4" gate="G$1" pin="2"/>
-<pinref part="GND13" gate="1" pin="GND"/>
-</segment>
-<segment>
 <pinref part="C8" gate="G$1" pin="2"/>
 <pinref part="GND14" gate="1" pin="GND"/>
@@
 <pinref part="GND32" gate="1" pin="GND"/>
 <pinref part="C18" gate="G$1" pin="2"/>
+</segment>
+<segment>
+<pinref part="GND13" gate="1" pin="GND"/>
+<pinref part="C4" gate="G$1" pin="2"/>
 </segment>
 </net>
@@
 <segment>
 <wire x1="261.62" y1="33.02" x2="264.16" y2="33.02" width="0.1524" layer="91"/>
-<wire x1="264.16" y1="33.02" x2="264.16" y2="38.1" width="0.1524" layer="91"/>
+<wire x1="264.16" y1="33.02" x2="264.16" y2="40.64" width="0.1524" layer="91"/>
 <pinref part="X1" gate="-1" pin="S"/>
 <pinref part="P+3" gate="1" pin="+5V"/>
@@
 <wire x1="365.76" y1="83.82" x2="373.38" y2="83.82" width="0.1524" layer="91"/>
 <wire x1="373.38" y1="83.82" x2="373.38" y2="81.28" width="0.1524" layer="91"/>
-<pinref part="C4" gate="G$1" pin="1"/>
 <wire x1="365.76" y1="83.82" x2="365.76" y2="81.28" width="0.1524" layer="91"/>
 <junction x="365.76" y="83.82"/>
 <pinref part="R5" gate="G$1" pin="1"/>
 <junction x="373.38" y="83.82"/>
-</segment>
-</net>
+<pinref part="C4" gate="G$1" pin="1"/>
+</segment>
+</net>

Commit message: Minor refinements
Andrea Zoppi
Parts:
- renumbered 1 to X4, 2 to X5, U$4 to X6
Changed lines of the file:
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@@
 <part name="GND12" library="supply1" deviceset="GND" device=""/>
 <part name="U3" library="st" deviceset="LD3985XX" device=""/>
-<part name="U$4" library="samtec" deviceset="FTSH-105" device=""/>
+<part name="X6" library="samtec" deviceset="FTSH-105" device=""/>
 <part name="+3V1" library="supply1" deviceset="+3V3" device=""/>
 <part name="GND4" library="supply1" deviceset="GND" device=""/>
@@
 <part name="C21" library="rcl" deviceset="C-EU" device="C0805" value="4u7"/>
 <part name="FRAME2" library="frames" deviceset="DINA3_L" device=""/>
-<part name="1" library="molex" deviceset="RJ45-43860" device=""/>
+<part name="X4" library="molex" deviceset="RJ45-43860" device=""/>
 <part name="JP1" library="misc" deviceset="PINHD-1X4" device=""/>
 <part name="GND1" library="supply1" deviceset="GND" device=""/>
-<part name="2" library="molex" deviceset="RJ45-43860" device=""/>
+<part name="X5" library="molex" deviceset="RJ45-43860" device=""/>
 <part name="JP2" library="misc" deviceset="PINHD-1X4" device=""/>
 <part name="GND19" library="supply1" deviceset="GND" device=""/>
@@
 <instance part="GND12" gate="1" x="187.96" y="71.12"/>
 <instance part="U3" gate="G$1" x="203.2" y="25.4"/>
-<instance part="U$4" gate="G$1" x="17.78" y="73.66"/>
+<instance part="X6" gate="G$1" x="17.78" y="73.66"/>
 <instance part="+3V1" gate="G$1" x="12.7" y="91.44"/>
 <instance part="GND4" gate="1" x="12.7" y="71.12"/>
@@
 <attribute name="DRAWING_NAME" x="304.8" y="19.05" size="2.54" layer="94" font="vector"/>
 </instance>
-<instance part="1" gate="G$1" x="99.06" y="25.4"/>
+<instance part="X4" gate="G$1" x="99.06" y="25.4"/>
 <instance part="JP1" gate="A" x="116.84" y="25.4"/>
 <instance part="GND1" gate="1" x="88.9" y="10.16"/>
-<instance part="2" gate="G$1" x="139.7" y="25.4"/>
+<instance part="X5" gate="G$1" x="139.7" y="25.4"/>
 <instance part="JP2" gate="A" x="157.48" y="25.4"/>
 <instance part="GND19" gate="1" x="129.54" y="10.16"/>
@@
 <segment>
 <wire x1="15.24" y1="83.82" x2="12.7" y2="83.82" width="0.1524" layer="91"/>
-<pinref part="U$4" gate="G$1" pin="3"/>
+<pinref part="X6" gate="G$1" pin="3"/>
 <wire x1="15.24" y1="76.2" x2="12.7" y2="76.2" width="0.1524" layer="91"/>
 <wire x1="12.7" y1="76.2" x2="12.7" y2="73.66" width="0.1524" layer="91"/>
-<pinref part="U$4" gate="G$1" pin="9"/>
+<pinref part="X6" gate="G$1" pin="9"/>
 <pinref part="GND4" gate="1" pin="GND"/>
 <junction x="12.7" y="76.2"/>
 <wire x1="15.24" y1="81.28" x2="12.7" y2="81.28" width="0.1524" layer="91"/>
 <wire x1="12.7" y1="81.28" x2="12.7" y2="83.82" width="0.1524" layer="91"/>
-<pinref part="U$4" gate="G$1" pin="5"/>
+<pinref part="X6" gate="G$1" pin="5"/>
 <junction x="12.7" y="81.28"/>
 <wire x1="12.7" y1="81.28" x2="12.7" y2="76.2" width="0.1524" layer="91"/>
@@
 <junction x="88.9" y="17.78"/>
 <junction x="88.9" y="20.32"/>
-<pinref part="1" gate="G$1" pin="6"/>
+<pinref part="X4" gate="G$1" pin="6"/>
 <pinref part="GND1" gate="1" pin="GND"/>
-<pinref part="1" gate="G$1" pin="7"/>
-<pinref part="1" gate="G$1" pin="8"/>
+<pinref part="X4" gate="G$1" pin="7"/>
+<pinref part="X4" gate="G$1" pin="8"/>
 <pinref part="JP1" gate="A" pin="4"/>
 <junction x="91.44" y="22.86"/>
-<pinref part="1" gate="G$1" pin="SHLD"/>
-<pinref part="1" gate="G$1" pin="P$1"/>
+<pinref part="X4" gate="G$1" pin="SHLD"/>
+<pinref part="X4" gate="G$1" pin="P$1"/>
 <wire x1="91.44" y1="15.24" x2="88.9" y2="15.24" width="0.1524" layer="91"/>
 <junction x="91.44" y="15.24"/>
@@
 <junction x="129.54" y="17.78"/>
 <junction x="129.54" y="20.32"/>
-<pinref part="2" gate="G$1" pin="6"/>
+<pinref part="X5" gate="G$1" pin="6"/>
 <pinref part="GND19" gate="1" pin="GND"/>
-<pinref part="2" gate="G$1" pin="7"/>
-<pinref part="2" gate="G$1" pin="8"/>
+<pinref part="X5" gate="G$1" pin="7"/>
+<pinref part="X5" gate="G$1" pin="8"/>
 <pinref part="JP2" gate="A" pin="4"/>
 <junction x="132.08" y="22.86"/>
-<pinref part="2" gate="G$1" pin="SHLD"/>
-<pinref part="2" gate="G$1" pin="P$1"/>
+<pinref part="X5" gate="G$1" pin="SHLD"/>
+<pinref part="X5" gate="G$1" pin="P$1"/>
 <wire x1="132.08" y1="15.24" x2="129.54" y2="15.24" width="0.1524" layer="91"/>
 <junction x="132.08" y="15.24"/>
@@
 <wire x1="15.24" y1="86.36" x2="12.7" y2="86.36" width="0.1524" layer="91"/>
 <wire x1="12.7" y1="86.36" x2="12.7" y2="88.9" width="0.1524" layer="91"/>
-<pinref part="U$4" gate="G$1" pin="1"/>
+<pinref part="X6" gate="G$1" pin="1"/>
 <pinref part="+3V1" gate="G$1" pin="+3V3"/>
 </segment>
@@
 <segment>
 <label x="33.02" y="86.36" size="1.778" layer="95"/>
-<pinref part="U$4" gate="G$1" pin="2"/>
+<pinref part="X6" gate="G$1" pin="2"/>
 <wire x1="30.48" y1="86.36" x2="33.02" y2="86.36" width="0.1524" layer="91"/>
 </segment>
@@
 <segment>
 <label x="33.02" y="83.82" size="1.778" layer="95"/>
-<pinref part="U$4" gate="G$1" pin="4"/>
+<pinref part="X6" gate="G$1" pin="4"/>
 <wire x1="30.48" y1="83.82" x2="33.02" y2="83.82" width="0.1524" layer="91"/>
 </segment>
@@
 <segment>
 <label x="33.02" y="81.28" size="1.778" layer="95"/>
-<pinref part="U$4" gate="G$1" pin="6"/>
+<pinref part="X6" gate="G$1" pin="6"/>
 <wire x1="30.48" y1="81.28" x2="33.02" y2="81.28" width="0.1524" layer="91"/>
 </segment>
@@
 <segment>
 <label x="33.02" y="78.74" size="1.778" layer="95"/>
-<pinref part="U$4" gate="G$1" pin="8"/>
+<pinref part="X6" gate="G$1" pin="8"/>
 <wire x1="30.48" y1="78.74" x2="33.02" y2="78.74" width="0.1524" layer="91"/>
 </segment>
@@
 <label x="88.9" y="27.94" size="1.778" layer="95" rot="MR0"/>
 <wire x1="91.44" y1="27.94" x2="114.3" y2="27.94" width="0.1524" layer="91"/>
-<pinref part="1" gate="G$1" pin="4"/>
+<pinref part="X4" gate="G$1" pin="4"/>
 <pinref part="JP1" gate="A" pin="2"/>
 <wire x1="88.9" y1="27.94" x2="91.44" y2="27.94" width="0.1524" layer="91"/>
@@
 <wire x1="132.08" y1="27.94" x2="129.54" y2="27.94" width="0.1524" layer="91"/>
 <label x="129.54" y="27.94" size="1.778" layer="95" rot="MR0"/>
-<pinref part="2" gate="G$1" pin="4"/>
+<pinref part="X5" gate="G$1" pin="4"/>
 <pinref part="JP2" gate="A" pin="2"/>
 <junction x="132.08" y="27.94"/>
@@
 <label x="88.9" y="25.4" size="1.778" layer="95" rot="MR0"/>
 <wire x1="91.44" y1="25.4" x2="114.3" y2="25.4" width="0.1524" layer="91"/>
-<pinref part="1" gate="G$1" pin="5"/>
+<pinref part="X4" gate="G$1" pin="5"/>
 <pinref part="JP1" gate="A" pin="3"/>
 <junction x="91.44" y="25.4"/>
@@
 <wire x1="132.08" y1="25.4" x2="129.54" y2="25.4" width="0.1524" layer="91"/>
 <label x="129.54" y="25.4" size="1.778" layer="95" rot="MR0"/>
-<pinref part="2" gate="G$1" pin="5"/>
+<pinref part="X5" gate="G$1" pin="5"/>
 <pinref part="JP2" gate="A" pin="3"/>
 <junction x="132.08" y="25.4"/>
@@
 <junction x="88.9" y="35.56"/>
 <junction x="88.9" y="33.02"/>
-<pinref part="1" gate="G$1" pin="3"/>
-<pinref part="1" gate="G$1" pin="2"/>
-<pinref part="1" gate="G$1" pin="1"/>
+<pinref part="X4" gate="G$1" pin="3"/>
+<pinref part="X4" gate="G$1" pin="2"/>
+<pinref part="X4" gate="G$1" pin="1"/>
 <pinref part="JP1" gate="A" pin="1"/>
 <junction x="91.44" y="30.48"/>
@@
 <junction x="129.54" y="35.56"/>
 <junction x="129.54" y="33.02"/>
-<pinref part="2" gate="G$1" pin="3"/>
-<pinref part="2" gate="G$1" pin="2"/>
-<pinref part="2" gate="G$1" pin="1"/>
+<pinref part="X5" gate="G$1" pin="3"/>
+<pinref part="X5" gate="G$1" pin="2"/>
+<pinref part="X5" gate="G$1" pin="1"/>
 <pinref part="JP2" gate="A" pin="1"/>
 <junction x="132.08" y="30.48"/>
@@
 <segment>
 <wire x1="30.48" y1="76.2" x2="33.02" y2="76.2" width="0.1524" layer="91"/>
-<pinref part="U$4" gate="G$1" pin="10"/>
+<pinref part="X6" gate="G$1" pin="10"/>
 <wire x1="33.02" y1="76.2" x2="33.02" y2="71.12" width="0.1524" layer="91"/>
 <wire x1="33.02" y1="71.12" x2="35.56" y2="71.12" width="0.1524" layer="91"/>
